Commit message: rviz

File: src/projeto/urdf/quadrotor_sonar.urdf.xacro (robot description, xacro)
@@ -16,6 +16,14 @@
     </xacro:sonar_sensor>
     <!-- Sonar front sensor -->
-    <xacro:sonar_sensor name="sonar_medida" parent="base_link" ros_topic="sonar_front" update_rate="10" min_range="0.2" max_range="3.0" field_of_view="2" ray_count="1">
+    <xacro:sonar_sensor name="sonar_medida0" parent="base_link" ros_topic="sonar_front" update_rate="10" min_range="0.2" max_range="5.0" field_of_view="2" ray_count="1">
       <origin xyz="0.1 0.0 0.12" rpy="0 0 0"/>
+    </xacro:sonar_sensor>
+    <!-- Sonar front sensor -->
+    <xacro:sonar_sensor name="sonar_medida1" parent="base_link" ros_topic="sonar_left" update_rate="10" min_range="0.2" max_range="5.0" field_of_view="2" ray_count="1">
+      <origin xyz="0.1 0.0 0.12" rpy="-1 0 0"/>
+    </xacro:sonar_sensor>
+    <!-- Sonar front sensor -->
+    <xacro:sonar_sensor name="sonar_medida2" parent="base_link" ros_topic="sonar_right" update_rate="10" min_range="0.2" max_range="5.0" field_of_view="2" ray_count="1">
+      <origin xyz="0.1 0.0 0.12" rpy="1 0 0"/>
     </xacro:sonar_sensor>
     <!-- Hokuyo UTM-30LX mounted upside down below the quadrotor body

Commit message: correcoes 1

File: src/projeto/urdf/quadrotor_sonar.urdf.xacro (robot description, xacro)
@@ -16,14 +16,14 @@
     </xacro:sonar_sensor>
     <!-- Sonar front sensor -->
-    <xacro:sonar_sensor name="sonar_medida0" parent="base_link" ros_topic="sonar_front" update_rate="10" min_range="0.2" max_range="5.0" field_of_view="2" ray_count="1">
+    <xacro:sonar_sensor name="sonar_medida0" parent="base_link" ros_topic="sonar_front" update_rate="15" min_range="0.2" max_range="3.0" field_of_view="1" ray_count="1">
       <origin xyz="0.1 0.0 0.12" rpy="0 0 0"/>
     </xacro:sonar_sensor>
-    <!-- Sonar front sensor -->
-    <xacro:sonar_sensor name="sonar_medida1" parent="base_link" ros_topic="sonar_left" update_rate="10" min_range="0.2" max_range="5.0" field_of_view="2" ray_count="1">
-      <origin xyz="0.1 0.0 0.12" rpy="-1 0 0"/>
+    <!-- Sonar left sensor -->
+    <xacro:sonar_sensor name="sonar_medida1" parent="base_link" ros_topic="sonar_left" update_rate="15" min_range="0.2" max_range="3.0" field_of_view="1" ray_count="1">
+      <origin xyz="0.1 0.0 0.12" rpy="0 0 -${30*M_PI/180}"/>
     </xacro:sonar_sensor>
-    <!-- Sonar front sensor -->
-    <xacro:sonar_sensor name="sonar_medida2" parent="base_link" ros_topic="sonar_right" update_rate="10" min_range="0.2" max_range="5.0" field_of_view="2" ray_count="1">
-      <origin xyz="0.1 0.0 0.12" rpy="1 0 0"/>
+    <!-- Sonar right sensor -->
+    <xacro:sonar_sensor name="sonar_medida2" parent="base_link" ros_topic="sonar_right" update_rate="15" min_range="0.2" max_range="3.0" field_of_view="1" ray_count="1">
+      <origin xyz="0.1 0.0 0.12" rpy="0 0 ${30*M_PI/180}"/>
     </xacro:sonar_sensor>
     <!-- Hokuyo UTM-30LX mounted upside down below the quadrotor body

Commit message: correcao simulador

File: src/projeto/urdf/quadrotor_sonar.urdf.xacro (robot description, xacro)
@@ -15,15 +15,19 @@
       <origin xyz="-0.15 0.0 0.0" rpy="0 ${90*M_PI/180} 0"/>
     </xacro:sonar_sensor>
-    <!-- Sonar front sensor -->
-    <xacro:sonar_sensor name="sonar_medida0" parent="base_link" ros_topic="sonar_front" update_rate="15" min_range="0.2" max_range="3.0" field_of_view="1" ray_count="1">
+    <!-- Sonar 1 sensor -->
+    <xacro:sonar_sensor name="sonar_medida0" parent="base_link" ros_topic="sensor1/dist" update_rate="10" min_range="0.2" max_range="1.5" field_of_view="1" ray_count="1">
       <origin xyz="0.1 0.0 0.12" rpy="0 0 0"/>
     </xacro:sonar_sensor>
-    <!-- Sonar left sensor -->
-    <xacro:sonar_sensor name="sonar_medida1" parent="base_link" ros_topic="sonar_left" update_rate="15" min_range="0.2" max_range="3.0" field_of_view="1" ray_count="1">
-      <origin xyz="0.1 0.0 0.12" rpy="0 0 -${30*M_PI/180}"/>
+    <!-- Sonar 2 sensor -${30*M_PI/180}-->
+    <xacro:sonar_sensor name="sonar_medida1" parent="base_link" ros_topic="sensor2/dist" update_rate="10" min_range="0.2" max_range="1.5" field_of_view="1" ray_count="1">
+      <origin xyz="0.1 0.0 0.12" rpy="0 0 0"/>
     </xacro:sonar_sensor>
-    <!-- Sonar right sensor -->
-    <xacro:sonar_sensor name="sonar_medida2" parent="base_link" ros_topic="sonar_right" update_rate="15" min_range="0.2" max_range="3.0" field_of_view="1" ray_count="1">
-      <origin xyz="0.1 0.0 0.12" rpy="0 0 ${30*M_PI/180}"/>
+    <!-- Sonar 3 sensor  ${30*M_PI/180}-->
+    <xacro:sonar_sensor name="sonar_medida2" parent="base_link" ros_topic="sensor3/dist" update_rate="10" min_range="0.2" max_range="1.5" field_of_view="1" ray_count="1">
+      <origin xyz="0.1 0.0 0.12" rpy="0 0 0"/>
+    </xacro:sonar_sensor>
+     <!-- Sonar 4 sensor -${30*M_PI/180}-->
+    <xacro:sonar_sensor name="sonar_medida3" parent="base_link" ros_topic="sensor4/dist" update_rate="10" min_range="0.2" max_range="1.5" field_of_view="1" ray_count="1">
+      <origin xyz="0.1 0.0 0.12" rpy="0 0 0"/>
     </xacro:sonar_sensor>
     <!-- Hokuyo UTM-30LX mounted upside down below the quadrotor body
